File: serafino l432kc.sch (KiCad schematic (older format))
At the start: 36 parts

Commit message: Battery charger
Parts:
- added U?: BQ24072RGT, Package_DFN_QFN:VQFN-16-1EP_3x3mm_P0.5mm_EP1.6x1.6mm, symbol Battery_Management:BQ24072RGT
Changed lines of the file:
@@
 Wire Wire Line
 	3700 3600 3700 3700
+$Comp
+L Battery_Management:BQ24072RGT U?
+U 1 1 5FD0D37B
+P 2950 4950
+F 0 "U?" H 2950 5731 50  0000 C CNN
+F 1 "BQ24072RGT" H 2950 5640 50  0000 C CNN
+F 2 "Package_DFN_QFN:VQFN-16-1EP_3x3mm_P0.5mm_EP1.6x1.6mm" H 3250 4400 50  0001 L CNN
+F 3 "http://www.ti.com/lit/ds/symlink/bq24072.pdf" H 3250 5150 50  0001 C CNN
+	1    2950 4950
+	1    0    0    -1
+$EndComp
 $EndSCHEMATC

Commit message: Simplificacion del Power Supply y eliminación del battery charger
Parts:
- removed C? (x2): 100nF, symbol Device:C_Small
- removed C?: 10uF, symbol Device:C_Small
- removed C?: 10pF, symbol Device:C_Small
- removed C? (x2): 22uF, symbol Device:C_Small
- removed C?: 4.7uF, symbol Device:C_Small
- removed J?: Conn_01x02, symbol Connector_Generic:Conn_01x02
- removed L?: 4.7uH, symbol Device:L_Small
- removed R?: 30.9k, symbol Device:R_Small
- removed R?: 10k, symbol Device:R_Small
- removed U?: MCP73831-2-OT, Package_TO_SOT_SMD:SOT-23-5, symbol Battery_Management:MCP73831-2-OT
- removed U?: TPS563207DRLR, Package_TO_SOT_SMD:SOT-23-6, symbol TPS563207DRLR:TPS563207DRLR
- removed U?: BQ24072RGT, Package_DFN_QFN:VQFN-16-1EP_3x3mm_P0.5mm_EP1.6x1.6mm, symbol Battery_Management:BQ24072RGT
- added C1: 1uF, symbol Device:C_Small
- added C3: 2.2uF, symbol Device:C_Small
- added J? (x2): Conn_01x10, symbol Connector_Generic:Conn_01x10
- added U1: AP2112K-3.3, Package_TO_SOT_SMD:SOT-23-5, symbol Regulator_Linear:AP2112K-3.3
- TC1: renamed from TC?; symbol TC2030-IDC:TC2030-IDC -> serafino-l432kc-rescue:TC2030-IDC-TC2030-IDC
- gave numbers to parts that had none: 22
Connections:
- net labels added: +VIN, PA15, PA5, PA8, PB4, PB5, PB6, PB7
- net labels removed: +12V, VBAT
- wire segments 125 -> 93
- no-connect marks 3 -> 4
Other:
- moved on the sheet: C10, C2, C4, C5, C6, C7, C8, C9, D1, J1, L1, R1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

Commit message: Pinout definition
Parts:
- removed J? (x2): Conn_01x10, symbol Connector_Generic:Conn_01x10
- added J2, J3: Conn_01x11, symbol Connector_Generic:Conn_01x11
Connections:
- net labels added: PA0, VHIGH
- wire segments 93 -> 97
Changed lines of the file:
@@
 Wire Wire Line
 	2350 1450 2350 1400
-Wire Wire Line
-	2350 1400 2600 1400
-Wire Wire Line
-	2700 1500 2600 1500
-Wire Wire Line
-	2600 1500 2600 1400
 $Comp
 L power:GND #PWR08
@@
 	1    0    0    -1
 $EndComp
-Connection ~ 2350 1400
 Wire Wire Line
 	1150 4900 1150 4800
 Wire Wire Line
 	1150 4800 1200 4800
-Wire Wire Line
-	2600 1400 2700 1400
-Connection ~ 2600 1400
 NoConn ~ 2150 7450
 Text GLabel 6500 4300 0    50   Input ~ 0
@@
 	7100 3100 7100 2900
 Wire Wire Line
-	750  1250 750  1400
-Wire Wire Line
-	750  1400 900  1400
-Wire Wire Line
-	2050 1400 2350 1400
+	2050 1400 2150 1400
 $Comp
-L power:+VIN #PWR?
+L power:+VIN #PWR0101
 U 1 1 5FE0AAFC
 P 750 1250
-F 0 "#PWR?" H 750 1100 50  0001 C CNN
+F 0 "#PWR0101" H 750 1100 50  0001 C CNN
 F 1 "+VIN" H 765 1423 50  0000 C CNN
 F 2 "" H 750 1250 50  0001 C CNN
@@
 	1    0    0    -1
 $EndComp
-Wire Wire Line
-	8350 3550 8950 3550
 Text GLabel 8950 3650 0    50   Input ~ 0
 SPI1_SCK
@@
 SPI1_MOSI
 $Comp
-L power:GND #PWR?
+L power:GND #PWR0102
 U 1 1 5FE261BD
-P 10950 3600
-F 0 "#PWR?" H 10950 3350 50  0001 C CNN
-F 1 "GND" H 10955 3427 50  0000 C CNN
-F 2 "" H 10950 3600 50  0001 C CNN
-F 3 "" H 10950 3600 50  0001 C CNN
-	1    10950 3600
+P 10650 3500
+F 0 "#PWR0102" H 10650 3250 50  0001 C CNN
+F 1 "GND" H 10655 3327 50  0000 C CNN
+F 2 "" H 10650 3500 50  0001 C CNN
+F 3 "" H 10650 3500 50  0001 C CNN
+	1    10650 3500
 	1    0    0    -1
 $EndComp
 Wire Wire Line
-	10950 3600 10950 3550
+	10650 3500 10650 3450
 Wire Wire Line
-	10450 3550 10950 3550
+	10150 3450 10650 3450
 $Comp
-L power:+3V3 #PWR?
+L power:+3V3 #PWR0103
 U 1 1 5FE29993
-P 8350 3400
-F 0 "#PWR?" H 8350 3250 50  0001 C CNN
-F 1 "+3V3" H 8365 3573 50  0000 C CNN
-F 2 "" H 8350 3400 50  0001 C CNN
-F 3 "" H 8350 3400 50  0001 C CNN
-	1    8350 3400
+P 8350 3250
+F 0 "#PWR0103" H 8350 3100 50  0001 C CNN
+F 1 "+3V3" H 8365 3423 50  0000 C CNN
+F 2 "" H 8350 3250 50  0001 C CNN
+F 3 "" H 8350 3250 50  0001 C CNN
+	1    8350 3250
 	1    0    0    -1
 $EndComp
-Wire Wire Line
-	8350 3400 8350 3550
 Text GLabel 6500 4800 0    50   Input ~ 0
 PB7
-Text GLabel 10450 3650 2    50   Input ~ 0
+Text GLabel 10150 3550 2    50   Input ~ 0
 PB7
 Text GLabel 6500 4700 0    50   Input ~ 0
@@
 Text GLabel 6500 4500 0    50   Input ~ 0
 PB4
-Text GLabel 10450 3750 2    50   Input ~ 0
+Text GLabel 10150 3650 2    50   Input ~ 0
 PB6
-Text GLabel 10450 3850 2    50   Input ~ 0
+Text GLabel 10150 3750 2    50   Input ~ 0
 PB5
-Text GLabel 10450 3950 2    50   Input ~ 0
+Text GLabel 10150 3850 2    50   Input ~ 0
 PB4
-Text GLabel 10450 4050 2    50   Input ~ 0
+Text GLabel 10150 3950 2    50   Input ~ 0
 SAI1_SCK_B
 Text GLabel 7500 4100 2    50   Input ~ 0
@@
 Text GLabel 7500 4800 2    50   Input ~ 0
 PA15
-Text GLabel 10450 4150 2    50   Input ~ 0
+Text GLabel 10150 4050 2    50   Input ~ 0
 PA15
-Text GLabel 10450 4250 2    50   Input ~ 0
+Text GLabel 10150 4150 2    50   Input ~ 0
 PA8
+Text GLabel 2150 950  1    50   Input ~ 0
+VHIGH
+Wire Wire Line
+	2150 950  2150 1400
+Connection ~ 2150 1400
+Wire Wire Line
+	2150 1400 2350 1400
+Text GLabel 10150 4350 2    50   Input ~ 0
+NRST
+Text GLabel 10150 4250 2    50   Input ~ 0
+VHIGH
+Wire Wire Line
+	2700 1400 2550 1400
+Connection ~ 2350 1400
+Wire Wire Line
+	2550 1500 2550 1400
+Connection ~ 2550 1400
+Wire Wire Line
+	2550 1400 2350 1400
+Wire Wire Line
+	2550 1500 2700 1500
+Wire Wire Line
+	750  1250 750  1400
+Wire Wire Line
+	750  1400 900  1400
 $Comp
-L Connector_Generic:Conn_01x10 J?
-U 1 1 5FE31848
+L Connector_Generic:Conn_01x11 J2
+U 1 1 5FD45AA3
 P 9150 3950
-F 0 "J?" H 9230 3942 50  0000 L CNN
-F 1 "Conn_01x10" H 9230 3851 50  0000 L CNN
+F 0 "J2" H 9230 3992 50  0000 L CNN
+F 1 "Conn_01x11" H 9230 3901 50  0000 L CNN
 F 2 "" H 9150 3950 50  0001 C CNN
 F 3 "~" H 9150 3950 50  0001 C CNN
@@
 $EndComp
 $Comp
-L Connector_Generic:Conn_01x10 J?
-U 1 1 5FE32CE6
-P 10250 4050
-F 0 "J?" H 10168 3325 50  0000 C CNN
-F 1 "Conn_01x10" H 10168 3416 50  0000 C CNN
-F 2 "" H 10250 4050 50  0001 C CNN
-F 3 "~" H 10250 4050 50  0001 C CNN
-	1    10250 4050
+L Connector_Generic:Conn_01x11 J3
+U 1 1 5FD47F36
+P 9950 3950
+F 0 "J3" H 9868 3225 50  0000 C CNN
+F 1 "Conn_01x11" H 9868 3316 50  0000 C CNN
+F 2 "" H 9950 3950 50  0001 C CNN
+F 3 "~" H 9950 3950 50  0001 C CNN
+	1    9950 3950
 	-1   0    0    1
 $EndComp
+$Comp
+L power:+VIN #PWR0104
+U 1 1 5FD50E68
+P 10700 4400
+F 0 "#PWR0104" H 10700 4250 50  0001 C CNN
+F 1 "+VIN" H 10715 4573 50  0000 C CNN
+F 2 "" H 10700 4400 50  0001 C CNN
+F 3 "" H 10700 4400 50  0001 C CNN
+	1    10700 4400
+	1    0    0    -1
+$EndComp
+Wire Wire Line
+	10700 4400 10700 4450
+Wire Wire Line
+	10700 4450 10150 4450
+Wire Wire Line
+	8350 3250 8350 3450
+Wire Wire Line
+	8350 3450 8950 3450
+Text GLabel 7500 3300 2    50   Input ~ 0
+PA0
+Text GLabel 8950 3550 0    50   Input ~ 0
+PA0
 $EndSCHEMATC

Commit message: PCB layout
Parts:
- removed J2, J3: Conn_01x11, symbol Connector_Generic:Conn_01x11
- added H1, H2, H3, H4: MountingHole_Pad, MountingHole:MountingHole_4.3mm_M4_Pad_Via, symbol Mechanical:MountingHole_Pad
- added J2, J3: Conn_01x13, Connector_PinHeader_2.54mm:PinHeader_1x13_P2.54mm_Vertical, symbol Connector_Generic:Conn_01x13
- added TP1: TestPoint, TestPoint:TestPoint_Bridge_Pitch2.0mm_Drill0.7mm, symbol Connector:TestPoint
- C1, C3: footprint (none) -> Capacitor_SMD:C_1206_3216Metric
- C10, C2, C4, C5, C6, C7, C9: footprint (none) -> Capacitor_SMD:C_0603_1608Metric
- C8: footprint (none) -> Capacitor_Tantalum_SMD:CP_EIA-1608-08_AVX-J
- D1: footprint (none) -> LED_SMD:LED_0603_1608Metric
- D2: footprint (none) -> Diode_SMD:D_SOD-123
- F1: footprint (none) -> Fuse:Fuse_1206_3216Metric
- FB1: footprint (none) -> Inductor_SMD:L_0805_2012Metric
- J1: footprint (none) -> Connector_USB:USB_Micro-B_Molex-105017-0001
- L1: footprint (none) -> Inductor_SMD:L_0603_1608Metric
- R1, R2: footprint (none) -> Resistor_SMD:R_0603_1608Metric
- SW1: footprint (none) -> Button_Switch_SMD:SW_Push_SPST_NO_Alps_SKRK
- SW2: footprint (none) -> Button_Switch_SMD:SW_SPDT_CK-JS102011SAQN
- TC1: footprint (none) -> Connector:Tag-Connect_TC2030-IDC-FP_2x03_P1.27mm_Vertical
- Y1: footprint (none) -> serafino l432kc:NX3215SA
Connections:
- net +3.3VA: now also J3.12 (Pin_12)
- net +3V3: now also J2.1 (Pin_1)
- net +5V: now also J2.13 (Pin_13)
- net +VIN: now also J3.1 (Pin_1)
- net GND: now also SW2.3 (C), H1.1, H2.1, H3.1, H4.1, J3.13 (Pin_13)
- net I2C1_SCL: now also J3.4 (Pin_4)
- net I2C1_SDA: now also J3.5 (Pin_5)
- net LED0: now also J2.12 (Pin_12)
- net NRST: now also J2.2 (Pin_2)
- net PA0: now also J2.3 (Pin_3)
- net PA15: now also J3.6 (Pin_6)
- net PA5: now also J2.8 (Pin_8)
- net PA8: now also J3.3 (Pin_3)
- net PB4: now also J3.8 (Pin_8)
- net PB5: now also J3.9 (Pin_9)
- net PB6: now also J3.10 (Pin_10)
- net PB7: now also J3.11 (Pin_11)
- net SAI1_FS_B: now also J2.7 (Pin_7)
- net SAI1_SCK_B: now also J3.7 (Pin_7)
- net SPI1_MISO: now also J2.9 (Pin_9)
- net SPI1_MOSI: now also J2.10 (Pin_10)
- net SPI1_SCK: now also J2.4 (Pin_4)
- net SPI1_SS: now also J2.11 (Pin_11)
- net USART2_RX: now also J2.6 (Pin_6)
- net USART2_TX: now also J2.5 (Pin_5)
- net VHIGH: now also J3.2 (Pin_2), TP1.1
- no-connect marks 4 -> 3

Commit message: Layout..
Parts:
- SW2: footprint Button_Switch_SMD:SW_SPDT_CK-JS102011SAQN -> Button_Switch_SMD:SW_DIP_SPSTx01_Slide_Copal_CHS-01A_W5.08mm_P1.27mm_JPin
Changed lines of the file:
@@
 F 0 "SW2" H 1950 7635 50  0000 C CNN
 F 1 "SW_SPDT" H 1950 7544 50  0000 C CNN
-F 2 "Button_Switch_SMD:SW_SPDT_CK-JS102011SAQN" H 1950 7350 50  0001 C CNN
+F 2 "Button_Switch_SMD:SW_DIP_SPSTx01_Slide_Copal_CHS-01A_W5.08mm_P1.27mm_JPin" H 1950 7350 50  0001 C CNN
 F 3 "~" H 1950 7350 50  0001 C CNN
 	1    1950 7350

Commit message: More layouts...
Parts:
- removed H1, H2, H3, H4: MountingHole_Pad, MountingHole:MountingHole_4.3mm_M4_Pad_Via, symbol Mechanical:MountingHole_Pad
- removed TP1: TestPoint, TestPoint:TestPoint_Bridge_Pitch2.0mm_Drill0.7mm, symbol Connector:TestPoint
- C1, C3: footprint Capacitor_SMD:C_1206_3216Metric -> Capacitor_SMD:C_0603_1608Metric
- C4, C5: footprint Capacitor_SMD:C_0603_1608Metric -> Capacitor_SMD:C_0402_1005Metric
- SW1: footprint Button_Switch_SMD:SW_Push_SPST_NO_Alps_SKRK -> Button_Switch_SMD:SW_Push_1P1T_NO_Vertical_Wuerth_434133025816
Changed lines of the file:
@@
 F 0 "C4" V 4471 4550 50  0000 C CNN
 F 1 "4.3pF" V 4562 4550 50  0000 C CNN
-F 2 "Capacitor_SMD:C_0603_1608Metric" H 4700 4550 50  0001 C CNN
+F 2 "Capacitor_SMD:C_0402_1005Metric" H 4700 4550 50  0001 C CNN
 F 3 "~" H 4700 4550 50  0001 C CNN
 	1    4700 4550
@@
 F 0 "C5" V 4850 4850 50  0000 C CNN
 F 1 "4.3pF" V 4950 4850 50  0000 C CNN
-F 2 "Capacitor_SMD:C_0603_1608Metric" H 4700 4850 50  0001 C CNN
+F 2 "Capacitor_SMD:C_0402_1005Metric" H 4700 4850 50  0001 C CNN
 F 3 "~" H 4700 4850 50  0001 C CNN
 	1    4700 4850
@@
 F 0 "SW1" V 2396 5052 50  0000 R CNN
 F 1 "SW_Push" V 2305 5052 50  0000 R CNN
-F 2 "Button_Switch_SMD:SW_Push_SPST_NO_Alps_SKRK" H 2350 5300 50  0001 C CNN
+F 2 "Button_Switch_SMD:SW_Push_1P1T_NO_Vertical_Wuerth_434133025816" H 2350 5300 50  0001 C CNN
 F 3 "~" H 2350 5300 50  0001 C CNN
 	1    2350 5100
@@
 F 0 "C3" H 3642 1596 50  0000 L CNN
 F 1 "2.2uF" H 3642 1505 50  0000 L CNN
-F 2 "Capacitor_SMD:C_1206_3216Metric" H 3550 1550 50  0001 C CNN
+F 2 "Capacitor_SMD:C_0603_1608Metric" H 3550 1550 50  0001 C CNN
 F 3 "~" H 3550 1550 50  0001 C CNN
 	1    3550 1550
@@
 F 0 "C1" H 2442 1596 50  0000 L CNN
 F 1 "1uF" H 2442 1505 50  0000 L CNN
-F 2 "Capacitor_SMD:C_1206_3216Metric" H 2350 1550 50  0001 C CNN
+F 2 "Capacitor_SMD:C_0603_1608Metric" H 2350 1550 50  0001 C CNN
 F 3 "~" H 2350 1550 50  0001 C CNN
 	1    2350 1550
@@
 Text GLabel 2150 950  1    50   Input ~ 0
 VHIGH
-Wire Wire Line
-	2150 950  2150 1100
 Connection ~ 2150 1400
 Wire Wire Line
@@
 Text GLabel 7500 3300 2    50   Input ~ 0
 PA0
-$Comp
-L Connector:TestPoint TP1
-U 1 1 5FD76707
-P 2450 850
-F 0 "TP1" V 2404 1038 50  0000 L CNN
-F 1 "TestPoint" V 2495 1038 50  0000 L CNN
-F 2 "TestPoint:TestPoint_Bridge_Pitch2.0mm_Drill0.7mm" H 2650 850 50  0001 C CNN
-F 3 "~" H 2650 850 50  0001 C CNN
-	1    2450 850
-	0    1    1    0
-$EndComp
-Wire Wire Line
-	2450 850  2450 1100
-Wire Wire Line
-	2450 1100 2150 1100
-Connection ~ 2150 1100
-Wire Wire Line
-	2150 1100 2150 1400
 Wire Wire Line
 	6900 3100 6800 3100
@@
 Wire Wire Line
 	2700 1400 2550 1400
-$Comp
-L Mechanical:MountingHole_Pad H1
-U 1 1 5FF05A28
-P 9750 5300
-F 0 "H1" V 9704 5450 50  0000 L CNN
-F 1 "MountingHole_Pad" V 9795 5450 50  0000 L CNN
-F 2 "MountingHole:MountingHole_4.3mm_M4_Pad_Via" H 9750 5300 50  0001 C CNN
-F 3 "~" H 9750 5300 50  0001 C CNN
-	1    9750 5300
-	0    1    1    0
-$EndComp
-$Comp
-L Mechanical:MountingHole_Pad H2
-U 1 1 5FF0858C
-P 9750 5500
-F 0 "H2" V 9704 5650 50  0000 L CNN
-F 1 "MountingHole_Pad" V 9795 5650 50  0000 L CNN
-F 2 "MountingHole:MountingHole_4.3mm_M4_Pad_Via" H 9750 5500 50  0001 C CNN
-F 3 "~" H 9750 5500 50  0001 C CNN
-	1    9750 5500
-	0    1    1    0
-$EndComp
-$Comp
-L Mechanical:MountingHole_Pad H3
-U 1 1 5FF08965
-P 9750 5700
-F 0 "H3" V 9704 5850 50  0000 L CNN
-F 1 "MountingHole_Pad" V 9795 5850 50  0000 L CNN
-F 2 "MountingHole:MountingHole_4.3mm_M4_Pad_Via" H 9750 5700 50  0001 C CNN
-F 3 "~" H 9750 5700 50  0001 C CNN
-	1    9750 5700
-	0    1    1    0
-$EndComp
-$Comp
-L Mechanical:MountingHole_Pad H4
-U 1 1 5FF08D38
-P 9750 5900
-F 0 "H4" V 9704 6050 50  0000 L CNN
-F 1 "MountingHole_Pad" V 9795 6050 50  0000 L CNN
-F 2 "MountingHole:MountingHole_4.3mm_M4_Pad_Via" H 9750 5900 50  0001 C CNN
-F 3 "~" H 9750 5900 50  0001 C CNN
-	1    9750 5900
-	0    1    1    0
-$EndComp
-Wire Wire Line
-	9650 5300 9550 5300
-Wire Wire Line
-	9550 5300 9550 5500
-Wire Wire Line
-	9550 5900 9650 5900
-Wire Wire Line
-	9650 5500 9550 5500
-Connection ~ 9550 5500
-Wire Wire Line
-	9550 5500 9550 5700
-Wire Wire Line
-	9650 5700 9550 5700
-Connection ~ 9550 5700
-Wire Wire Line
-	9550 5700 9550 5900
-$Comp
-L power:GND #PWR01
-U 1 1 5FF1CA95
-P 9550 6100
-F 0 "#PWR01" H 9550 5850 50  0001 C CNN
-F 1 "GND" H 9555 5927 50  0000 C CNN
-F 2 "" H 9550 6100 50  0001 C CNN
-F 3 "" H 9550 6100 50  0001 C CNN
-	1    9550 6100
-	1    0    0    -1
-$EndComp
-Wire Wire Line
-	9550 6100 9550 5900
-Connection ~ 9550 5900
+Wire Wire Line
+	2150 950  2150 1400
 $EndSCHEMATC
